File: Hardware/A111_Pulsed_Radar_Breakout.brd (EAGLE design)
At the start: 33 x 39.4 mm, 45 parts, among them J4 RASPBERRYPI-26-PIN-GPIO, U1 A111, U2 1.8V, U4 TXB0108DQSR, Y1 26MHz

Commit message: Replaces SparkFun silk with SparkFun silk with flame, grounds, 1.8V voltage regulator
Parts:
- removed LOGO4: SFE_LOGO_FLAME.2_INCH, SparkFun-Aesthetics:SFE_LOGO_FLAME_.2
- LOGO1, LOGO3: value SFE_LOGO_NAME.1_INCH -> SFE_LOGO_NAME_FLAME.1_INCH; device SparkFun-Aesthetics:SFE_LOGO_NAME_.1 -> SparkFun-Aesthetics:SFE_LOGO_NAME_FLAME_.1
- moved LOGO1 1.52 mm to (16.5, 35.3)
- moved LOGO3 1.52 mm to (16.5, 35.3)
- moved LOGO2 1.30 mm to (3.17, 8.51), flipped to the top
- moved FD2 1.27 mm to (0.64, 38.7)
- moved FD3 1.27 mm to (0.64, 38.7)
- moved H1 1.27 mm to (2.54, 36.8)
- moved H2 1.27 mm to (30.5, 36.8)
- moved U$1 1.27 mm to (4.19, 33.1)
- moved U$9 1.27 mm to (28.8, 33.1)
- moved Y1 1.27 mm to (21.6, 25.4)
- moved FD1 1.27 mm to (31.8, 6.35)
- moved FD4 1.27 mm to (31.8, 6.35)
- moved J2 1.27 mm to (25.4, 6.35)
- moved J4 1.27 mm to (31.8, 3.81)
- moved C1 1.27 mm to (11.4, 26.7)
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Connections:
- net GND: now also U2.2
