File: Hardware/A111_Pulsed_Radar_Breakout.sch (EAGLE design)
At the start: 27 parts, among them J4 RASPBERRYPI-26-PIN-GPIO, U1 A111, U2 1.8V, U4 TXB0108DQSR, Y1 26MHz

Commit message: Adds SparkFun logo to the underside, migrates all parts to SparkFun libraries.
Parts:
- J4: device A111_Radar:RASPBERRYPI-26-PIN-GPIO -> SparkFun-Connectors:RASPBERRYPI-26-PIN-GPIO
Other:
- note added: "40 pin is backwards compatible with 26 pin header."
- moved on the sheet: C1, C10, C2, C3, C4, C5, C6, C7, C8, C9, R1, U1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
